Commit message: Consolidate volcaniarm into delta_arms_description; remove old package
Move the volcaniarm urdf, meshes (under meshes/volcaniarm/), launch, and world into
delta_arms_description and rewrite the package:// mesh paths and launch package refs.
Verified the volcaniarm still spawns and loads its meshes from the new package, then
removed the now-unused volcaniarm_description package.

Co-Authored-By: Claude Opus 4.8 (1M context) <noreply@anthropic.com>

File: src/delta_arms_description/urdf/volcaniarm.urdf (robot description, URDF)
Before this commit: robot volcaniarm, 24 links, 23 joints
Links:
- link base_link: geometry collision mesh filename=package://delta_arms_description/meshes/volcaniarm/base_lin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; visual mesh filename=package://delta_arms_description/meshes/volcaniarm/base_lin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
- link camera_link: geometry collision mesh filename=package://delta_arms_description/meshes/volcaniarm/camera_l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; visual mesh filename=package://delta_arms_description/meshes/volcaniarm/camera_l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
- link camera_mount_linear_link: geometry collision mesh filename=package://delta_arms_description/meshes/volcaniarm/camera_m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; visual mesh filename=package://delta_arms_description/meshes/volcaniarm/camera_m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
- link camera_mount_rev_link: geometry collision mesh filename=package://delta_arms_description/meshes/volcaniarm/camera_m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; visual mesh filename=package://delta_arms_description/meshes/volcaniarm/camera_m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
- link fl_caster_wheel_link: geometry collision mesh filename=package://delta_arms_description/meshes/volcaniarm/fl_caste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; visual mesh filename=package://delta_arms_description/meshes/volcaniarm/fl_caste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
- link fl_caster_wheel_mount_link: geometry collision mesh filename=package://delta_arms_description/meshes/volcaniarm/fl_caste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; visual mesh filename=package://delta_arms_description/meshes/volcaniarm/fl_caste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
- link fl_table_leg_link: geometry collision mesh filename=package://delta_arms_description/meshes/volcaniarm/fl_table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; visual mesh filename=package://delta_arms_description/meshes/volcaniarm/fl_table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
- link fr_caster_wheel_link: geometry collision mesh filename=package://delta_arms_description/meshes/volcaniarm/fr_caste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; visual mesh filename=package://delta_arms_description/meshes/volcaniarm/fr_caste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
- link fr_caster_wheel_mount_link: geometry collision mesh filename=package://delta_arms_description/meshes/volcaniarm/fr_caste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; visual mesh filename=package://delta_arms_description/meshes/volcaniarm/fr_caste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
- link fr_table_leg_link: geometry collision mesh filename=package://delta_arms_description/meshes/volcaniarm/fr_table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; visual mesh filename=package://delta_arms_description/meshes/volcaniarm/fr_table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
- link rl_caster_wheel_link: geometry collision mesh filename=package://delta_arms_description/meshes/volcaniarm/rl_caste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; visual mesh filename=package://delta_arms_description/meshes/volcaniarm/rl_caste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
- link rl_caster_wheel_mount_link: geometry collision mesh filename=package://delta_arms_description/meshes/volcaniarm/rl_caste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; visual mesh filename=package://delta_arms_description/meshes/volcaniarm/rl_caste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
- link rl_table_leg_link: geometry collision mesh filename=package://delta_arms_description/meshes/volcaniarm/rl_table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; visual mesh filename=package://delta_arms_description/meshes/volcaniarm/rl_table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
- link rr_caster_wheel_link: geometry collision mesh filename=package://delta_arms_description/meshes/volcaniarm/rr_caste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; visual mesh filename=package://delta_arms_description/meshes/volcaniarm/rr_caste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
- link rr_caster_wheel_mount_link: geometry collision mesh filename=package://delta_arms_description/meshes/volcaniarm/rr_caste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; visual mesh filename=package://delta_arms_description/meshes/volcaniarm/rr_caste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
- link rr_table_leg_link: geometry collision mesh filename=package://delta_arms_description/meshes/volcaniarm/rr_table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; visual mesh filename=package://delta_arms_description/meshes/volcaniarm/rr_table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
- link volcaniarm_base_link: geometry collision mesh filename=package://delta_arms_description/meshes/volcaniarm/volcania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; visual mesh filename=package://delta_arms_description/meshes/volcaniarm/volcania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
- link volcaniarm_left_arm_link: geometry collision mesh filename=package://delta_arms_description/meshes/volcaniarm/volcania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; visual mesh filename=package://delta_arms_description/meshes/volcaniarm/volcania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
- link volcaniarm_left_elbow_link: geometry collision mesh filename=package://delta_arms_description/meshes/volcaniarm/volcania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; visual mesh filename=package://delta_arms_description/meshes/volcaniarm/volcania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
- link volcaniarm_right_arm_link: geometry collision mesh filename=package://delta_arms_description/meshes/volcaniarm/volcania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; visual mesh filename=package://delta_arms_description/meshes/volcaniarm/volcania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
- link volcaniarm_right_elbow_link: geometry collision mesh filename=package://delta_arms_description/meshes/volcaniarm/volcania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; visual mesh filename=package://delta_arms_description/meshes/volcaniarm/volcania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
