Commit message: fivebar_linkage: drop the table, promote linkage mount to base_link
Remove the table top (the old base_link) entirely and rename linkage_base_link ->
base_link, so the robot is just the base + the two chains. Fold the removed
linkage_base_joint transform into world_to_base (xyz 0.218 0 0.96, rpy 0 pi 0) so the
linkage keeps its pose, and rename the mesh linkage_base_link.STL -> base_link.STL.

Verified: single base_link, clean tree, spawns ~0.96 m above ground, loop closes.

Co-Authored-By: Claude Opus 4.8 (1M context) <noreply@anthropic.com>

File: src/delta_arms_description/urdf/fivebar_linkage.urdf (robot description, URDF)
Before this commit: robot fivebar_linkage, 9 links, 8 joints
Links:
- removed link linkage_base_link
- link base_link: mass 5.4796 -> 5.2358
Joints:
- removed joint linkage_base_joint
- joint Chain1_1: parent linkage_base_link -> base_link
- joint Chain2_1: parent linkage_base_link -> base_link
- joint world_to_base: origin xyz=0 0 0.98 rpy=0 0 3.14159 -> xyz=0.218 0 0.96 rpy=0 3.14159 0
