Commit message: Restructure into description + bringup packages; drop URDF generators
Split delta_arms_description into two packages:
- closed_loop_description: URDFs, Gazebo worlds, meshes (what the robots are)
- closed_loop_bringup: launch files (how to start them)
Rename reflects that all three robots (5-bar + deltas) are closed-loop mechanisms.
Update package:// mesh refs, launch get_package_share_directory calls, and the
ros_gz_bridge args accordingly. Launch is now: ros2 launch closed_loop_bringup <robot>.launch.py

Also remove the scripts/ delta URDF generators (the URDFs are now static files) and
rewrite the README for the two-package layout: updated repo structure, usage, and
implementation-guide paths; reduced em-dash usage.

Co-Authored-By: Claude Opus 4.8 (1M context) <noreply@anthropic.com>

File: src/closed_loop_description/urdf/3dof_delta.urdf (robot description, URDF)
Before this commit: robot deltaarm_4dof, 38 links, 37 joints
Links:
- removed link Chain4_bottom_link
- removed link Chain4_cl_v1
- removed link Chain4_cl_v2
- removed link Chain4_dummy
- removed link Chain4_tip
- removed link Chain4_top_link
- removed link Chain4_top_v1
- removed link Chain4_top_v2
- removed link tool_holder
- link Chain1_forearm: mass 0.15 -> 0.08; geometry visual mesh filename=package://closed_loop_description/meshes/PARA_ENGINEER/Unte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 scale=0.001 0.001 0.001
- link Chain1_link_1: mass 0.5 -> 0.3; geometry visual mesh filename=package://closed_loop_description/meshes/PARA_ENGINEER/Ober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 scale=0.001 0.001 0.001
- link Chain2_forearm: mass 0.15 -> 0.08; geometry visual mesh filename=package://closed_loop_description/meshes/PARA_ENGINEER/Unte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 scale=0.001 0.001 0.001
- link Chain2_link_1: mass 0.5 -> 0.3; geometry visual mesh filename=package://closed_loop_description/meshes/PARA_ENGINEER/Ober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 scale=0.001 0.001 0.001
- link Chain3_forearm: mass 0.15 -> 0.08; geometry visual mesh filename=package://closed_loop_description/meshes/PARA_ENGINEER/Unte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 scale=0.001 0.001 0.001
- link Chain3_link_1: mass 0.5 -> 0.3; geometry visual mesh filename=package://closed_loop_description/meshes/PARA_ENGINEER/Ober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 scale=0.001 0.001 0.001
- link base_link: geometry visual mesh filename=package://closed_loop_description/meshes/PARA_ENGINEER/Kopf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 scale=0.001 0.001 0.001
- link tool0: mass 0.2 -> 0.3; geometry visual mesh filename=package://closed_loop_description/meshes/PARA_ENGINEER/Werk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 scale=0.001 0.001 0.001
Joints:
- removed joint Chain4_1
- removed joint Chain4_4
- removed joint Chain4_cl_A
- removed joint Chain4_cl_B
- removed joint Chain4_cl_C
- removed joint Chain4_tip_joint
- removed joint Chain4_top_A
- removed joint Chain4_top_B
- removed joint Chain4_top_C
- joint Chain1_1: origin xyz=0.250000 0.000000 0 rpy=0 0 0.000000 -> xyz=0.041700 0.000000 0 rpy=0 0 0.000000
- joint Chain1_cl_A: origin xyz=0.070000 0.000000 0 rpy=0 2.187225 0.000000 -> xyz=0.027600 0.000000 0 rpy=0 2.140009 0.000000; parent tool_holder -> tool0
- joint Chain1_tip_joint: origin xyz=0.960000 0 0 rpy=0 0 0 -> xyz=0.166800 0 0 rpy=0 0 0
- joint Chain1_top_A: origin xyz=0.375000 0 0 rpy=0 2.187225 0 -> xyz=0.075800 0 0 rpy=0 2.140009 0
- joint Chain2_1: origin xyz=-0.125000 0.216506 0 rpy=0 0 2.094395 -> xyz=-0.020850 0.036113 0 rpy=0 0 2.094395
- joint Chain2_cl_A: origin xyz=-0.035000 0.060622 0 rpy=0 2.187225 2.094395 -> xyz=-0.013800 0.023902 0 rpy=0 2.140009 2.094395; parent tool_holder -> tool0
- joint Chain2_tip_joint: origin xyz=0.960000 0 0 rpy=0 0 0 -> xyz=0.166800 0 0 rpy=0 0 0
- joint Chain2_top_A: origin xyz=0.375000 0 0 rpy=0 2.187225 0 -> xyz=0.075800 0 0 rpy=0 2.140009 0
- joint Chain3_1: origin xyz=-0.125000 -0.216506 0 rpy=0 0 4.188790 -> xyz=-0.020850 -0.036113 0 rpy=0 0 4.188790
- joint Chain3_cl_A: origin xyz=-0.035000 -0.060622 0 rpy=0 2.187225 4.188790 -> xyz=-0.013800 -0.023902 0 rpy=0 2.140009 4.188790; parent tool_holder -> tool0
- joint Chain3_tip_joint: origin xyz=0.960000 0 0 rpy=0 0 0 -> xyz=0.166800 0 0 rpy=0 0 0
- joint Chain3_top_A: origin xyz=0.375000 0 0 rpy=0 2.187225 0 -> xyz=0.075800 0 0 rpy=0 2.140009 0
- joint platform_x: limit lower=-0.7 upper=0.7 effort=99999.0 velocity=99999.0 -> lower=-0.5 upper=0.5 effort=99999.0 velocity=99999.0; origin xyz=0 0 -0.783310 rpy=0 0 0 -> xyz=0 0 -0.140500 rpy=0 0 0
- joint platform_y: limit lower=-0.7 upper=0.7 effort=99999.0 velocity=99999.0 -> lower=-0.5 upper=0.5 effort=99999.0 velocity=99999.0
- joint platform_z: child tool_holder -> tool0; limit lower=-0.7 upper=0.7 effort=99999.0 velocity=99999.0 -> lower=-0.5 upper=0.5 effort=99999.0 velocity=99999.0
- joint world_to_base: origin xyz=0 0 1.600000 rpy=0 0 0 -> xyz=0 0 1.000000 rpy=0 0 0

File: src/closed_loop_description/urdf/4dof_delta.urdf (robot description, URDF)
Before this commit: robot deltaarm_3dof, 29 links, 28 joints
Links:
- added link Chain4_bottom_link, mass 0.2; visual mesh filename=package://closed_loop_description/meshes/A_00036/Teleskopwe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 scale=0.001 0.001 0.001
- added link Chain4_cl_v1, mass 0.01
- added link Chain4_cl_v2, mass 0.01
- added link Chain4_dummy, mass 0.01
- added link Chain4_tip, mass 0.01
- added link Chain4_top_link, mass 0.2; visual mesh filename=package://closed_loop_description/meshes/A_00036/Teleskopwe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 scale=0.001 0.001 0.001
- added link Chain4_top_v1, mass 0.01
- added link Chain4_top_v2, mass 0.01
- added link tool_holder, mass 0.4; visual mesh filename=package://closed_loop_description/meshes/A_00036/Werkzeugtr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 scale=0.001 0.001 0.001
- link Chain1_forearm: mass 0.08 -> 0.15; geometry visual mesh filename=package://closed_loop_description/meshes/A_00036/Unterarm.s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 scale=0.001 0.001 0.001
- link Chain1_link_1: mass 0.3 -> 0.5; geometry visual mesh filename=package://closed_loop_description/meshes/A_00036/Oberarm.stl scale=0.001 0.001 0.001
- link Chain2_forearm: mass 0.08 -> 0.15; geometry visual mesh filename=package://closed_loop_description/meshes/A_00036/Unterarm.s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 scale=0.001 0.001 0.001
- link Chain2_link_1: mass 0.3 -> 0.5; geometry visual mesh filename=package://closed_loop_description/meshes/A_00036/Oberarm.stl scale=0.001 0.001 0.001
- link Chain3_forearm: mass 0.08 -> 0.15; geometry visual mesh filename=package://closed_loop_description/meshes/A_00036/Unterarm.s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 scale=0.001 0.001 0.001
- link Chain3_link_1: mass 0.3 -> 0.5; geometry visual mesh filename=package://closed_loop_description/meshes/A_00036/Oberarm.stl scale=0.001 0.001 0.001
- link base_link: geometry visual mesh filename=package://closed_loop_description/meshes/A_00036/Kopfplatte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 scale=0.001 0.001 0.001
- link tool0: mass 0.3 -> 0.2; geometry visual mesh filename=package://closed_loop_description/meshes/A_00036/Flansch.stl scale=0.001 0.001 0.001
Joints:
- added joint Chain4_1: type revolute, parent tool_holder, child tool0, origin xyz=0 0 0 rpy=0 0 0, axis 0 0 1, limit lower=-7.0 upper=7.0 effort=42.0 velocity=785.0
- added joint Chain4_4: type prismatic, parent Chain4_top_link, child Chain4_bottom_link, origin xyz=0 0 -0.783310 rpy=0 0 0, axis 0 0 -1, limit lower=0.0 upper=0.7 effort=1000.0 velocity=10.0
- added joint Chain4_cl_A: type revolute, parent tool0, child Chain4_cl_v1, origin xyz=0 0 0 rpy=0 0 0, axis 1 0 0, limit lower=-3.141592653589793 upper=3.141592653589793 effort=99999.0 velocity=99999.0
- added joint Chain4_cl_B: type revolute, parent Chain4_cl_v1, child Chain4_cl_v2, origin xyz=0 0 0 rpy=0 0 0, axis 0 1 0, limit lower=-3.141592653589793 upper=3.141592653589793 effort=99999.0 velocity=99999.0
- added joint Chain4_cl_C: type revolute, parent Chain4_cl_v2, child Chain4_dummy, origin xyz=0 0 0 rpy=0 0 0, axis 0 0 1, limit lower=-3.141592653589793 upper=3.141592653589793 effort=99999.0 velocity=99999.0
- added joint Chain4_tip_joint: type fixed, parent Chain4_bottom_link, child Chain4_tip, origin xyz=0 0 0 rpy=0 0 0
- added joint Chain4_top_A: type revolute, parent base_link, child Chain4_top_v1, origin xyz=0 0 0 rpy=0 0 0, axis 1 0 0, limit lower=-3.141592653589793 upper=3.141592653589793 effort=99999.0 velocity=99999.0
- added joint Chain4_top_B: type revolute, parent Chain4_top_v1, child Chain4_top_v2, origin xyz=0 0 0 rpy=0 0 0, axis 0 1 0, limit lower=-3.141592653589793 upper=3.141592653589793 effort=99999.0 velocity=99999.0
- added joint Chain4_top_C: type revolute, parent Chain4_top_v2, child Chain4_top_link, origin xyz=0 0 0 rpy=0 0 0, axis 0 0 1, limit lower=-3.141592653589793 upper=3.141592653589793 effort=99999.0 velocity=99999.0
- joint Chain1_1: origin xyz=0.041700 0.000000 0 rpy=0 0 0.000000 -> xyz=0.250000 0.000000 0 rpy=0 0 0.000000
- joint Chain1_cl_A: origin xyz=0.027600 0.000000 0 rpy=0 2.140009 0.000000 -> xyz=0.070000 0.000000 0 rpy=0 2.187225 0.000000; parent tool0 -> tool_holder
- joint Chain1_tip_joint: origin xyz=0.166800 0 0 rpy=0 0 0 -> xyz=0.960000 0 0 rpy=0 0 0
- joint Chain1_top_A: origin xyz=0.075800 0 0 rpy=0 2.140009 0 -> xyz=0.375000 0 0 rpy=0 2.187225 0
- joint Chain2_1: origin xyz=-0.020850 0.036113 0 rpy=0 0 2.094395 -> xyz=-0.125000 0.216506 0 rpy=0 0 2.094395
- joint Chain2_cl_A: origin xyz=-0.013800 0.023902 0 rpy=0 2.140009 2.094395 -> xyz=-0.035000 0.060622 0 rpy=0 2.187225 2.094395; parent tool0 -> tool_holder
- joint Chain2_tip_joint: origin xyz=0.166800 0 0 rpy=0 0 0 -> xyz=0.960000 0 0 rpy=0 0 0
- joint Chain2_top_A: origin xyz=0.075800 0 0 rpy=0 2.140009 0 -> xyz=0.375000 0 0 rpy=0 2.187225 0
- joint Chain3_1: origin xyz=-0.020850 -0.036113 0 rpy=0 0 4.188790 -> xyz=-0.125000 -0.216506 0 rpy=0 0 4.188790
- joint Chain3_cl_A: origin xyz=-0.013800 -0.023902 0 rpy=0 2.140009 4.188790 -> xyz=-0.035000 -0.060622 0 rpy=0 2.187225 4.188790; parent tool0 -> tool_holder
- joint Chain3_tip_joint: origin xyz=0.166800 0 0 rpy=0 0 0 -> xyz=0.960000 0 0 rpy=0 0 0
- joint Chain3_top_A: origin xyz=0.075800 0 0 rpy=0 2.140009 0 -> xyz=0.375000 0 0 rpy=0 2.187225 0
- joint platform_x: limit lower=-0.5 upper=0.5 effort=99999.0 velocity=99999.0 -> lower=-0.7 upper=0.7 effort=99999.0 velocity=99999.0; origin xyz=0 0 -0.140500 rpy=0 0 0 -> xyz=0 0 -0.783310 rpy=0 0 0
- joint platform_y: limit lower=-0.5 upper=0.5 effort=99999.0 velocity=99999.0 -> lower=-0.7 upper=0.7 effort=99999.0 velocity=99999.0
- joint platform_z: child tool0 -> tool_holder; limit lower=-0.5 upper=0.5 effort=99999.0 velocity=99999.0 -> lower=-0.7 upper=0.7 effort=99999.0 velocity=99999.0
- joint world_to_base: origin xyz=0 0 1.000000 rpy=0 0 0 -> xyz=0 0 1.600000 rpy=0 0 0

File: src/closed_loop_description/urdf/fivebar_linkage.urdf (robot description, URDF)
Before this commit: robot fivebar_linkage, 8 links, 7 joints
Links:
- link Chain1_link_1: geometry collision mesh filename=package://closed_loop_description/meshes/fivebar_linkage/Ch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; visual mesh filename=package://closed_loop_description/meshes/fivebar_linkage/Ch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
- link Chain1_link_2: geometry collision mesh filename=package://closed_loop_description/meshes/fivebar_linkage/Ch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; visual mesh filename=package://closed_loop_description/meshes/fivebar_linkage/Ch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
- link Chain2_link_1: geometry collision mesh filename=package://closed_loop_description/meshes/fivebar_linkage/Ch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; visual mesh filename=package://closed_loop_description/meshes/fivebar_linkage/Ch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
- link Chain2_link_2: geometry collision mesh filename=package://closed_loop_description/meshes/fivebar_linkage/Ch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; visual mesh filename=package://closed_loop_description/meshes/fivebar_linkage/Ch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
- link base_link: geometry collision mesh filename=package://closed_loop_description/meshes/fivebar_linkage/ba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; visual mesh filename=package://closed_loop_description/meshes/fivebar_linkage/ba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
