Commit message: Add closed-loop MoveIt+Gazebo pipeline; wire up fivebar_linkage
Port the HIT-Robotics joint_state_transformer pipeline so MoveIt can plan
motions for closed-loop parallel robots and execute them in Gazebo.

- Vendor the kinematics engine as submodules (forked urdfdom/urdfdom_headers,
  pinocchio 3.9 rebuilt against the fork, robot_model, joint_state_transformer).
- Single-source-of-truth xacro per robot: flag-gated macros (constraints / moveit
  phantom chain / ros2_control) mirroring the existing sim/gazebo split.
- fivebar_linkage end-to-end: gz_ros2_control on the active joints, the transformer
  doing IK (MoveIt tool pose -> motors) and FK (fill passives for RViz), a MoveIt
  config package, and a bringup launch. Includes an in-process orange ghost preview
  of the full closed-loop arm before execution.

Verified headlessly: a tool-pose goal drives the Gazebo motors to the predicted
angles; full /joint_states reconstructs the closed loop.

Co-Authored-By: Claude Opus 4.8 (1M context) <noreply@anthropic.com>

File: src/closed_loop_description/urdf/fivebar_linkage.gazebo.xacro (robot description, xacro)
@@ -3,4 +3,58 @@
 <!-- Included by fivebar_linkage.urdf.xacro via <xacro:include>. -->
 <robot xmlns:xacro="http://www.ros.org/wiki/xacro">
+  <!-- ===================================================================
+       Loop-closure helper frames (Gazebo/DetachableJoint only).
+       These are the leaves the DetachableJoint welds together; they live here (not in
+       the shared base tree) because the robot_model and MoveIt renders close the loop
+       differently and would see Chain1_closure as a dangling free joint.
+       Both frames are coincident at q=0 so the weld locks with zero relative motion. =-->
+  <!-- Massless tip frame fixed to the right arm at the physical closure point -->
+  <link name="Chain2_tip">
+    <inertial>
+      <origin xyz="0 0 0" rpy="0 0 0" />
+      <mass value="0.001" />
+      <inertia ixx="1e-6" ixy="0" ixz="0" iyy="1e-6" iyz="0" izz="1e-6" />
+    </inertial>
+    <visual>
+      <origin xyz="0 0 0" rpy="0 0 0" />
+      <geometry><sphere radius="0.008" /></geometry>
+      <material name="tip_green"><color rgba="0.95 0.75 0.10 1.0" /></material>
+    </visual>
+    <collision>
+      <origin xyz="0 0 0" rpy="0 0 0" />
+      <geometry><sphere radius="0.008" /></geometry>
+    </collision>
+  </link>
+  <joint name="Chain2_tip_joint" type="fixed">
+    <origin xyz="0 0 0.6225" rpy="0 0 0" />
+    <parent link="Chain2_link_2" />
+    <child link="Chain2_tip" />
+  </joint>
+  <!-- Closure dummy link: URDF-tree leaf on the left arm, DetachableJoint target.
+       rpy=(1.8398,0,0) rotates it so its frame matches Chain2_tip at q=0. -->
+  <link name="Chain1_dummy">
+    <inertial>
+      <origin xyz="0 0 0" rpy="0 0 0" />
+      <mass value="0.001" />
+      <inertia ixx="1e-6" ixy="0" ixz="0" iyy="1e-6" iyz="0" izz="1e-6" />
+    </inertial>
+    <visual>
+      <origin xyz="0 0 0" rpy="0 0 0" />
+      <geometry><sphere radius="0.008" /></geometry>
+      <material name="closure_purple"><color rgba="0.95 0.75 0.10 1.0" /></material>
+    </visual>
+    <collision>
+      <origin xyz="0 0 0" rpy="0 0 0" />
+      <geometry><sphere radius="0.008" /></geometry>
+    </collision>
+  </link>
+  <joint name="Chain1_closure" type="revolute">
+    <origin xyz="0 0 0.6225" rpy="1.8398 0 0" />
+    <parent link="Chain1_link_2" />
+    <child link="Chain1_dummy" />
+    <axis xyz="1 0 0" />
+    <limit lower="-3.14" upper="3.14" effort="0" velocity="10" />
+    <dynamics damping="0.1" friction="0.0" />
+  </joint>
   <!-- Prevent Gazebo from merging this fixed joint so DetachableJoint can find the link -->
   <gazebo reference="Chain2_tip_joint">
@@ -15,41 +69,44 @@
     </plugin>
   </gazebo>
-  <gazebo>
-    <plugin filename="libgz-sim-joint-position-controller-system.so"
-            name="gz::sim::systems::JointPositionController">
-      <joint_name>Chain1_1</joint_name>
-      <topic>/fivebar_linkage/Chain1_1/cmd_pos</topic>
-      <p_gain>10</p_gain>
-      <i_gain>1</i_gain>
-      <d_gain>1</d_gain>
-      <i_max>5</i_max>
-      <i_min>-5</i_min>
-      <cmd_max>10</cmd_max>
-      <cmd_min>-10</cmd_min>
-    </plugin>
-  </gazebo>
-  <gazebo>
-    <plugin filename="libgz-sim-joint-position-controller-system.so"
-            name="gz::sim::systems::JointPositionController">
-      <joint_name>Chain2_1</joint_name>
-      <topic>/fivebar_linkage/Chain2_1/cmd_pos</topic>
-      <p_gain>10</p_gain>
-      <i_gain>1</i_gain>
-      <d_gain>1</d_gain>
-      <i_max>5</i_max>
-      <i_min>-5</i_min>
-      <cmd_max>10</cmd_max>
-      <cmd_min>-10</cmd_min>
-    </plugin>
-  </gazebo>
-  <!-- Joint state publisher: broadcasts all joint positions back to ROS2 -->
-  <gazebo>
-    <plugin filename="libgz-sim-joint-state-publisher-system.so"
-            name="gz::sim::systems::JointStatePublisher">
-      <!-- publish ONLY the actuated joints, to mimic real encoders;
-           the passive joints are not measured on real hardware -->
-      <joint_name>Chain1_1</joint_name>
-      <joint_name>Chain2_1</joint_name>
-    </plugin>
-  </gazebo>
+  <!-- Open-loop control path (pure-sim only). When ros2_control:=true these are OFF and the
+       active joints are driven by gz_ros2_control / the actuated_joint_trajectory_controller
+       instead, so they are not double-commanded. -->
+  <xacro:unless value="$(arg ros2_control)">
+    <gazebo>
+      <plugin filename="libgz-sim-joint-position-controller-system.so"
+              name="gz::sim::systems::JointPositionController">
+        <joint_name>Chain1_1</joint_name>
+        <topic>/fivebar_linkage/Chain1_1/cmd_pos</topic>
+        <p_gain>10</p_gain>
+        <i_gain>1</i_gain>
+        <d_gain>1</d_gain>
+        <i_max>5</i_max>
+        <i_min>-5</i_min>
+        <cmd_max>10</cmd_max>
+        <cmd_min>-10</cmd_min>
+      </plugin>
+    </gazebo>
+    <gazebo>
+      <plugin filename="libgz-sim-joint-position-controller-system.so"
+              name="gz::sim::systems::JointPositionController">
+        <joint_name>Chain2_1</joint_name>
+        <topic>/fivebar_linkage/Chain2_1/cmd_pos</topic>
+        <p_gain>10</p_gain>
+        <i_gain>1</i_gain>
+        <d_gain>1</d_gain>
+        <i_max>5</i_max>
+        <i_min>-5</i_min>
+        <cmd_max>10</cmd_max>
+        <cmd_min>-10</cmd_min>
+      </plugin>
+    </gazebo>
+    <!-- Joint state publisher: broadcasts the actuated joints back to ROS2 (mimics encoders) -->
+    <gazebo>
+      <plugin filename="libgz-sim-joint-state-publisher-system.so"
+              name="gz::sim::systems::JointStatePublisher">
+        <joint_name>Chain1_1</joint_name>
+        <joint_name>Chain2_1</joint_name>
+      </plugin>
+    </gazebo>
+  </xacro:unless>
 </robot>

File: src/closed_loop_description/urdf/fivebar_linkage.urdf.xacro (robot description, xacro)
@@ -39,5 +39,5 @@
         name="">
         <color
-          rgba="0.25 0.25 0.25 1.0" />
+          rgba="0.75 0.78 0.82 1.0" />
       </material>
     </visual>
@@ -79,5 +79,5 @@
         name="">
         <color
-          rgba="0.25 0.25 0.25 1.0" />
+          rgba="0.75 0.78 0.82 1.0" />
       </material>
     </visual>
@@ -140,5 +140,5 @@
         name="">
         <color
-          rgba="0.25 0.25 0.25 1.0" />
+          rgba="0.75 0.78 0.82 1.0" />
       </material>
     </visual>
@@ -201,5 +201,5 @@
         name="">
         <color
-          rgba="0.25 0.25 0.25 1.0" />
+          rgba="0.75 0.78 0.82 1.0" />
       </material>
     </visual>
@@ -262,5 +262,5 @@
         name="">
         <color
-          rgba="0.25 0.25 0.25 1.0" />
+          rgba="0.75 0.78 0.82 1.0" />
       </material>
     </visual>
@@ -297,96 +297,43 @@
   </joint>
   <!-- ===================================================================
-       5-BAR LINKAGE CLOSURE
-       FK at q=0 (all revolute joints at zero):
-         Cumulative Rx to left arm link  : 2.2217 rad
-         Cumulative Rx to right arm link : -2.2217 rad  (mirror)
+       5-BAR LINKAGE CLOSURE  (FK reference at q=0, all revolute joints zero)
          Left arm origin in base_link    : (0.071,  0.4953, -0.3918)
          Right arm origin in base_link   : (0.075, -0.4953, -0.3918)
-         Arm z-axis (left)  in base_link : [0, -0.7956, -0.6059]
-         Arm z-axis (right) in base_link : [0, +0.7956, -0.6059]
-         Tip length L = 0.4953/0.7956   = 0.6225 m  (left arm CoM at L/2 = 0.311 m confirms)
-         Closure point in base_link      : (~0.073, 0, -0.769)
-         Chain1_closure rpy_r = 4.0615 - 2.2217 = 1.8398 rad  (aligns dummy with right tip frame)
+         Tip length L = 0.4953/0.7956   = 0.6225 m
+         Closure point in base_link      : (~0.073, 0, -0.769)   <- X_EE_PLANE = 0.073
+       The two distal links (Chain1_link_2, Chain2_link_2) meet at this closure point.
+       HOW THE LOOP IS CLOSED depends on the render (see flag-gated includes below):
+         - Gazebo  (sim):         DetachableJoint weld + helper frames (fivebar_linkage.gazebo.xacro)
+         - robot_model (constraints): two spherical <constraint>s to tool0 (fivebar_linkage.constraints.xacro)
+         - MoveIt  (planning):    phantom tool chain only          (fivebar_linkage.moveit.xacro)
+       The base tree above is shared by all renders and stays parser-agnostic.
        =================================================================== -->
-  <!-- Massless tip frame fixed to the right arm at the physical closure point -->
-  <link name="Chain2_tip">
-    <inertial>
-      <origin xyz="0 0 0" rpy="0 0 0" />
-      <mass value="0.001" />
-      <inertia ixx="1e-6" ixy="0" ixz="0" iyy="1e-6" iyz="0" izz="1e-6" />
-    </inertial>
-    <visual>
-      <origin xyz="0 0 0" rpy="0 0 0" />
-      <geometry>
-        <sphere radius="0.008" />
-      </geometry>
-      <material name="tip_green">
-        <color rgba="0.95 0.75 0.10 1.0" />
-      </material>
-    </visual>
-    <collision>
-      <origin xyz="0 0 0" rpy="0 0 0" />
-      <geometry>
-        <sphere radius="0.008" />
-      </geometry>
-    </collision>
-  </link>
-  <joint name="Chain2_tip_joint" type="fixed">
-    <origin xyz="0 0 0.6225" rpy="0 0 0" />
-    <parent link="Chain2_link_2" />
-    <child link="Chain2_tip" />
-  </joint>
-  <!-- Closure dummy link: URDF-tree leaf on the left arm, DetachableJoint target -->
-  <link name="Chain1_dummy">
-    <inertial>
-      <origin xyz="0 0 0" rpy="0 0 0" />
-      <mass value="0.001" />
-      <inertia ixx="1e-6" ixy="0" ixz="0" iyy="1e-6" iyz="0" izz="1e-6" />
-    </inertial>
-    <visual>
-      <origin xyz="0 0 0" rpy="0 0 0" />
-      <geometry>
-        <sphere radius="0.008" />
-      </geometry>
-      <material name="closure_purple">
-        <color rgba="0.95 0.75 0.10 1.0" />
-      </material>
-    </visual>
-    <collision>
-      <origin xyz="0 0 0" rpy="0 0 0" />
-      <geometry>
-        <sphere radius="0.008" />
-      </geometry>
-    </collision>
-  </link>
-  <!-- rpy=(1.8398,0,0) rotates Chain1_dummy so its world frame matches
-       Chain2_tip at q=0 → DetachableJoint locks with zero relative rotation -->
-  <joint name="Chain1_closure" type="revolute">
-    <origin xyz="0 0 0.6225" rpy="1.8398 0 0" />
-    <parent link="Chain1_link_2" />
-    <child link="Chain1_dummy" />
-    <axis xyz="1 0 0" />
-    <limit lower="-3.14" upper="3.14" effort="0" velocity="10" />
-    <dynamics damping="0.1" friction="0.0" />
-  </joint>
-  <!-- DetachableJoint: auto-attaches at launch, closing the 5-bar loop.
-       parent = Chain2_tip  (right chain leaf)
-       child  = Chain1_dummy  (left chain leaf)
-       Both frames are coincident at q=0, so no snap/impulse at attach time. -->
   <!-- ===================================================================
-       JOINT POSITION CONTROLLERS
-       Actuated joints of the 5-bar linkage:
-         - Chain1_1   (motor 1)
-         - Chain2_1  (motor 2)
-       Passive joints are driven by the linkage constraint:
-         - Chain1_2, Chain2_2, Chain1_closure
+       Single source of truth: one kinematic tree, four orthogonal add-on renders,
+       each gated by its own arg and split into its own macro file (mirrors the
+       existing sim/gazebo split). Each launch context renders with the flags it needs:
+         Gazebo:      sim:=true ros2_control:=true
+         MoveIt:      planning:=true
+         transformer: planning:=true constraints:=true   (constraints need tool0 from the phantom chain)
        =================================================================== -->
-  <!-- Sim vs. real separation: the kinematics above are shared by both. The Gazebo
-       system plugins and DetachableJoint loop closures are simulation-only, so they live
-       in a separate file included only when sim:=true. For real-hardware bringup
-       (sim:=false) a fivebar_linkage.ros2_control.xacro will be included here instead (added later). -->
-  <xacro:arg name="sim" default="true"/>
+  <xacro:arg name="sim"          default="true"/>
+  <xacro:arg name="ros2_control" default="false"/>
+  <xacro:arg name="planning"     default="false"/>
+  <xacro:arg name="constraints"  default="false"/>
+  <!-- Gazebo system plugins + DetachableJoint loop closure (+ closure helper frames) -->
   <xacro:if value="$(arg sim)">
     <xacro:include filename="fivebar_linkage.gazebo.xacro"/>
   </xacro:if>
+  <!-- ros2_control hardware interface on the active joints (gz_ros2_control in sim) -->
+  <xacro:if value="$(arg ros2_control)">
+    <xacro:include filename="fivebar_linkage.ros2_control.xacro"/>
+  </xacro:if>
+  <!-- MoveIt phantom planning chain to tool0 -->
+  <xacro:if value="$(arg planning)">
+    <xacro:include filename="fivebar_linkage.moveit.xacro"/>
+  </xacro:if>
+  <!-- Closed-loop <constraint> elements + transmissions for robot_model -->
+  <xacro:if value="$(arg constraints)">
+    <xacro:include filename="fivebar_linkage.constraints.xacro"/>
+  </xacro:if>
 </robot>
