Commit message: Fix delta_4dof IK (drop redundant column constraint); per-robot RViz; clean node shutdown
- delta_4dof was moving the wrong way / aborting from MoveIt: the central telescopic
  column was constrained to tool0 in addition to the 3 legs, adding a redundant passive
  DOF (nullspace) that made the Levenberg-Marquardt IK flaky (e.g. upward EE goals failed
  to converge). The EE pose is fully set by the 3 legs (translation) + the actuated flange
  Chain4_1 (rotation), so the column constraint is removed; the column still simulates in
  Gazebo via its own DetachableJoint. IK now converges 13/13 across the workspace and the
  Gazebo EE tracks the planned direction.
- Per-robot RViz configs (fivebar_linkage / delta_3dof / delta_4dof) with EE interactive
  marker + TF axis sizes scaled to each robot; each launch loads its own.
- description_publisher / transformer_with_preview: use rclpy.try_shutdown() so Ctrl+C/SIGINT
  exits cleanly instead of raising "rcl_shutdown already called".

Co-Authored-By: Claude Opus 4.8 (1M context) <noreply@anthropic.com>

File: src/closed_loop_description/urdf/4dof_delta.constraints.xacro (robot description, xacro)
@@ -38,8 +38,9 @@
     <child link="tool_holder"/><child_origin xyz="-0.035000 -0.060622 0"/>
   </constraint>
-  <!-- central telescopic column tip coincides with tool0 (the rotating flange) -->
-  <constraint name="Chain4_ee_constraint" type="spherical_joint">
-    <parent link="Chain4_bottom_link"/><parent_origin xyz="0 0 0"/>
-    <child link="tool0"/><child_origin xyz="0 0 0"/>
-  </constraint>
+  <!-- NOTE: the central telescopic column is intentionally NOT constrained here. The EE pose is
+       fully determined by the 3 legs (platform translation) + the actuated flange Chain4_1
+       (rotation); constraining the column too adds redundant passive DOF (a nullspace) that makes
+       the Levenberg-Marquardt IK flaky/non-convergent. The column is still simulated in Gazebo
+       (its own DetachableJoint) and follows physically. -->
+  <!-- (no Chain4 column constraint) -->
 </robot>
