Commit message: Fix delta_4dof MoveIt execution: reorder trajectory joints to model order; gate central column sim-only
MoveIt sends the executed trajectory joint_names in its own order ([Chain4_1, platform_x,
platform_y, platform_z]), but the upstream transformer assigns positions by ascending model
index, so every value landed on the wrong joint (cyclic shift) -- the real cause of the 4dof
wrong-axis / 'going down' behavior. transformer_with_preview now reorders each incoming
trajectory (execute + preview) to model order (no-op for 3dof/fivebar). Also gate the central
telescopic column sim-only so it is not a free chain in the solver/MoveIt model.

Co-Authored-By: Claude Opus 4.8 (1M context) <noreply@anthropic.com>

File: src/closed_loop_description/urdf/4dof_delta.urdf.xacro (robot description, xacro)
@@ -367,102 +367,13 @@
     <dynamics damping="0.1" friction="0.0"/>
   </joint>
-  <!-- ===================== central telescopic shaft (4th-axis column) ===================== -->
-  <link name="Chain4_top_link">
-    <visual>
-      <origin xyz="0 0 0" rpy="0 0 0"/>
-      <geometry>
-        <mesh filename="package://closed_loop_description/meshes/A_00036/Teleskopwelle_oben.stl" scale="0.001 0.001 0.001"/>
-      </geometry>
-      <material name="mat_shaft">
-        <color rgba="0.45 0.45 0.50 1.0"/>
-      </material>
-    </visual>
-    <inertial>
-      <origin xyz="0 0 0" rpy="0 0 0"/>
-      <mass value="0.2"/>
-      <inertia ixx="0.0005" ixy="0" ixz="0" iyy="0.0005" iyz="0" izz="0.0002"/>
-    </inertial>
-  </link>
-  <link name="Chain4_bottom_link">
-    <visual>
-      <origin xyz="0 0 0" rpy="0 0 0"/>
-      <geometry>
-        <mesh filename="package://closed_loop_description/meshes/A_00036/Teleskopwelle_unten.stl" scale="0.001 0.001 0.001"/>
-      </geometry>
-      <material name="mat_shaft">
-        <color rgba="0.45 0.45 0.50 1.0"/>
-      </material>
-    </visual>
-    <inertial>
-      <origin xyz="0 0 0" rpy="0 0 0"/>
-      <mass value="0.2"/>
-      <inertia ixx="0.0005" ixy="0" ixz="0" iyy="0.0005" iyz="0" izz="0.0002"/>
-    </inertial>
-  </link>
-  <link name="Chain4_tip">
-    <inertial>
-      <origin xyz="0 0 0" rpy="0 0 0"/>
-      <mass value="0.01"/>
-      <inertia ixx="1e-05" ixy="0" ixz="0" iyy="1e-05" iyz="0" izz="1e-05"/>
-    </inertial>
-  </link>
-  <link name="Chain4_top_v1">
-    <inertial>
-      <origin xyz="0 0 0" rpy="0 0 0"/>
-      <mass value="0.01"/>
-      <inertia ixx="1e-05" ixy="0" ixz="0" iyy="1e-05" iyz="0" izz="1e-05"/>
-    </inertial>
-  </link>
-  <link name="Chain4_top_v2">
-    <inertial>
-      <origin xyz="0 0 0" rpy="0 0 0"/>
-      <mass value="0.01"/>
-      <inertia ixx="1e-05" ixy="0" ixz="0" iyy="1e-05" iyz="0" izz="1e-05"/>
-    </inertial>
-  </link>
-  <joint name="Chain4_top_A" type="revolute">
-    <parent link="base_link"/>
-    <child link="Chain4_top_v1"/>
-    <origin xyz="0 0 0" rpy="0 0 0"/>
-    <axis xyz="1 0 0"/>
-    <limit effort="99999.0" lower="-3.141592653589793" upper="3.141592653589793" velocity="99999.0"/>
-    <dynamics damping="0.02" friction="0.0"/>
-  </joint>
-  <joint name="Chain4_top_B" type="revolute">
-    <parent link="Chain4_top_v1"/>
-    <child link="Chain4_top_v2"/>
-    <origin xyz="0 0 0" rpy="0 0 0"/>
-    <axis xyz="0 1 0"/>
-    <limit effort="99999.0" lower="-3.141592653589793" upper="3.141592653589793" velocity="99999.0"/>
-    <dynamics damping="0.02" friction="0.0"/>
-  </joint>
-  <joint name="Chain4_top_C" type="revolute">
-    <parent link="Chain4_top_v2"/>
-    <child link="Chain4_top_link"/>
-    <origin xyz="0 0 0" rpy="0 0 0"/>
-    <axis xyz="0 0 1"/>
-    <limit effort="99999.0" lower="-3.141592653589793" upper="3.141592653589793" velocity="99999.0"/>
-    <dynamics damping="0.02" friction="0.0"/>
-  </joint>
-  <joint name="Chain4_4" type="prismatic">
-    <parent link="Chain4_top_link"/>
-    <child link="Chain4_bottom_link"/>
-    <origin xyz="0 0 -0.783310" rpy="0 0 0"/>
-    <axis xyz="0 0 -1"/>
-    <limit effort="1000.0" lower="0.0" upper="0.7" velocity="10.0"/>
-    <dynamics damping="0.2" friction="0.0"/>
-  </joint>
-  <joint name="Chain4_tip_joint" type="fixed">
-    <parent link="Chain4_bottom_link"/>
-    <child link="Chain4_tip"/>
-    <origin xyz="0 0 0" rpy="0 0 0"/>
-  </joint>
   <!-- ===================================================================
        Single source of truth: one kinematic tree + flag-gated add-on macros (mirrors the
-       sim/gazebo split). The platform (platform_x/y/z -> tool_holder -> Chain4_1 -> tool0) and the
-       central telescopic column are already in the base tree; base_link -> tool0 IS the MoveIt
-       planning chain. The closure helper chains below (Chain*_cl_*, Chain*_dummy) are
-       DetachableJoint targets, sim-only; robot_model closes the loops with spherical <constraint>s
-       anchored on the forearms / Chain4_bottom_link (4dof_delta.constraints.xacro) instead.
+       sim/gazebo split). The platform (platform_x/y/z -> tool_holder -> Chain4_1 -> tool0) IS the
+       MoveIt planning chain base_link -> tool0. Everything below (the central telescopic column +
+       the closure helper chains) is Gazebo/DetachableJoint-only and is gated sim-only. robot_model
+       closes the loop with spherical <constraint>s on the 3 legs (4dof_delta.constraints.xacro) and
+       the EE rotation is the actuated flange Chain4_1, so the column is not needed for the solve.
+       (Left in the solver model as a free chain, it would drift past its limits and break the IK's
+       isStateValid() check -> "Levenberg-Marquardt failed to converge".)
          Gazebo:      sim:=true ros2_control:=true
          MoveIt:      (base tree; sim:=false)
@@ -473,4 +384,95 @@
   <xacro:arg name="constraints"  default="false"/>
   <xacro:if value="$(arg sim)">
+  <!-- ===================== central telescopic shaft (4th-axis column) ===================== -->
+  <link name="Chain4_top_link">
+    <visual>
+      <origin xyz="0 0 0" rpy="0 0 0"/>
+      <geometry>
+        <mesh filename="package://closed_loop_description/meshes/A_00036/Teleskopwelle_oben.stl" scale="0.001 0.001 0.001"/>
+      </geometry>
+      <material name="mat_shaft">
+        <color rgba="0.45 0.45 0.50 1.0"/>
+      </material>
+    </visual>
+    <inertial>
+      <origin xyz="0 0 0" rpy="0 0 0"/>
+      <mass value="0.2"/>
+      <inertia ixx="0.0005" ixy="0" ixz="0" iyy="0.0005" iyz="0" izz="0.0002"/>
+    </inertial>
+  </link>
+  <link name="Chain4_bottom_link">
+    <visual>
+      <origin xyz="0 0 0" rpy="0 0 0"/>
+      <geometry>
+        <mesh filename="package://closed_loop_description/meshes/A_00036/Teleskopwelle_unten.stl" scale="0.001 0.001 0.001"/>
+      </geometry>
+      <material name="mat_shaft">
+        <color rgba="0.45 0.45 0.50 1.0"/>
+      </material>
+    </visual>
+    <inertial>
+      <origin xyz="0 0 0" rpy="0 0 0"/>
+      <mass value="0.2"/>
+      <inertia ixx="0.0005" ixy="0" ixz="0" iyy="0.0005" iyz="0" izz="0.0002"/>
+    </inertial>
+  </link>
+  <link name="Chain4_tip">
+    <inertial>
+      <origin xyz="0 0 0" rpy="0 0 0"/>
+      <mass value="0.01"/>
+      <inertia ixx="1e-05" ixy="0" ixz="0" iyy="1e-05" iyz="0" izz="1e-05"/>
+    </inertial>
+  </link>
+  <link name="Chain4_top_v1">
+    <inertial>
+      <origin xyz="0 0 0" rpy="0 0 0"/>
+      <mass value="0.01"/>
+      <inertia ixx="1e-05" ixy="0" ixz="0" iyy="1e-05" iyz="0" izz="1e-05"/>
+    </inertial>
+  </link>
+  <link name="Chain4_top_v2">
+    <inertial>
+      <origin xyz="0 0 0" rpy="0 0 0"/>
+      <mass value="0.01"/>
+      <inertia ixx="1e-05" ixy="0" ixz="0" iyy="1e-05" iyz="0" izz="1e-05"/>
+    </inertial>
+  </link>
+  <joint name="Chain4_top_A" type="revolute">
+    <parent link="base_link"/>
+    <child link="Chain4_top_v1"/>
+    <origin xyz="0 0 0" rpy="0 0 0"/>
+    <axis xyz="1 0 0"/>
+    <limit effort="99999.0" lower="-3.141592653589793" upper="3.141592653589793" velocity="99999.0"/>
+    <dynamics damping="0.02" friction="0.0"/>
+  </joint>
+  <joint name="Chain4_top_B" type="revolute">
+    <parent link="Chain4_top_v1"/>
+    <child link="Chain4_top_v2"/>
+    <origin xyz="0 0 0" rpy="0 0 0"/>
+    <axis xyz="0 1 0"/>
+    <limit effort="99999.0" lower="-3.141592653589793" upper="3.141592653589793" velocity="99999.0"/>
+    <dynamics damping="0.02" friction="0.0"/>
+  </joint>
+  <joint name="Chain4_top_C" type="revolute">
+    <parent link="Chain4_top_v2"/>
+    <child link="Chain4_top_link"/>
+    <origin xyz="0 0 0" rpy="0 0 0"/>
+    <axis xyz="0 0 1"/>
+    <limit effort="99999.0" lower="-3.141592653589793" upper="3.141592653589793" velocity="99999.0"/>
+    <dynamics damping="0.02" friction="0.0"/>
+  </joint>
+  <joint name="Chain4_4" type="prismatic">
+    <parent link="Chain4_top_link"/>
+    <child link="Chain4_bottom_link"/>
+    <origin xyz="0 0 -0.783310" rpy="0 0 0"/>
+    <axis xyz="0 0 -1"/>
+    <limit effort="1000.0" lower="0.0" upper="0.7" velocity="10.0"/>
+    <dynamics damping="0.2" friction="0.0"/>
+  </joint>
+  <joint name="Chain4_tip_joint" type="fixed">
+    <parent link="Chain4_bottom_link"/>
+    <child link="Chain4_tip"/>
+    <origin xyz="0 0 0" rpy="0 0 0"/>
+  </joint>
   <link name="Chain4_dummy">
     <inertial>
